File: Schematic/mek6802D5/mek6802D5.kicad_sch (KiCad schematic)
At the start: 3 parts, among them U1 74LS244, U2 74LS244

Commit message: Adding to schematic
Parts:
- removed unit 2 of U1
- removed unit 2 of U2
- added C1, C2: C, symbol Device:C
- added J2: Conn_02x06_Odd_Even, symbol Connector_Generic:Conn_02x06_Odd_Even
- added R1, R2, R3, R5: 7K, symbol Device:R
- added R4: 4.7K, symbol Device:R
- added U10: 74LS244, symbol 0.MekLib:74LS244
- added U13: 2316 ROM, symbol 0.MekLib:ROM
- added U3: 47LS245, symbol 0.MekLib:74LS245
- added U4: 74LS00, symbol 74xx:74LS00
- added U5: MC6802, Package_DIP:DIP-40_W15.24mm, symbol 0.MekLib:6802
- added U6: MC68A21, Package_DIP:DIP-40_W15.24mm, symbol 0.MekLib:MC6821
- added U7, U8: MC2114, symbol 0.MekLib:MC2114
- added Y1: Crystal, symbol Device:Crystal
Connections:
- net MR is gone; now on net Ø2(E): TP1. (D7)
- net BA: now also U10.5 (O2b); no longer TP1. (D7)
- net BA0: now also U13.8 (A0), U5.9 (A0), U7.5 (A0), U8.5 (A0)
- net BA1: now also U13.7 (A1), U5.10 (A1), U7.6 (A1), U8.6 (A1)
- net BA10: now also J2.4 (Pin_4), J2.6 (Pin_6), U5.19 (A10)
- net BA11: now also U5.20 (A11)
- net BA12: now also U5.22 (A12)
- net BA13: now also U5.23 (A13)
- net BA14: now also U5.24 (A14)
- net BA15: now also U5.25 (A15)
- net BA2: now also U13.6 (A2), U5.11 (A2), U7.7 (A2), U8.7 (A2)
- net BA3: now also U13.5 (A3), U5.12 (A3), U7.4 (A3), U8.4 (A3)
- net BA4: now also U13.4 (A4), U5.13 (A4), U7.3 (A4), U8.3 (A4)
- net BA5: now also U13.3 (A5), U5.14 (A5), U7.2 (A5), U8.2 (A5)
- net BA6: now also U13.2 (A6), U5.15 (A6), U7.1 (A6), U8.1 (A6)
- net BA7: now also U13.1 (A7), U5.16 (A7), U7.17 (A7), U8.17 (A7)
- net BA8: now also U13.23 (A8), U5.17 (A8), U7.16 (A8), U8.16 (A8)
- net BA9: now also U13.22 (A9), U5.18 (A9), U7.15 (A9), U8.15 (A9)
- net E(Ø2): now also U10.18 (O0a); no longer TP1. (D7)
- net GND: now also U10.1 (OEa), U10.11 (I0b), U10.13 (I1b), U10.19 (OEb), U10.6 (I2a), U10.8 (I3a)
- net R/~{W}: now also U10.16 (O1a), U10.4 (I1a), U3.1 (A->B), U7.10 (~{W}), U8.10 (~{W})
- net YMA: now also U10.3 (O3b); no longer TP1. (D7)
- net ~{HALT}: now also R2.2, U5.2 (~{HALT})
- net ~{IRQ}: now also R3.2, U5.4 (~{IRQ})
- net ~{NMI}: now also R1.2, U5.6 (~{NMI})
- net ~{RESET}: now also R4.2, U5.40 (~{RESET})
- net Ø2(E): now reaches TP1. (D7)
- net Ø2(E): now also U10.2 (I0a), U4.5
- new net: U4.6, U7.8 (~{S}), U8.8 (~{S})
- new net: TP1. (D7), U3.2 (A0)
- new net: TP1. (D7), U3.3 (A1)
- new net: TP1. (D7), U3.4 (A2)
- new net: TP1. (D7), U3.5 (A3)
- new net: TP1. (D7), U3.6 (A4)
- new net: TP1. (D7), U3.7 (A5)
- new net: TP1. (D7), U3.8 (A6)
- new net: TP1. (D7), U3.9 (A7)
- new net: U4.11, U4.4
- new net: C1.2, C2.1
- new net: C2.2, U5.38 (XTAL), Y1.1
- new net: J2.3 (Pin_3), U13.19
- new net: J2.5 (Pin_5), J2.7 (Pin_7), U13.20
- new net: J2.8 (Pin_8), U13.18
- new net: J2.9 (Pin_9), U13.21
- new net: C1.1, U5.39 (EXTAL), Y1.2
- new net: U4.12, U4.13
- new net +12V: J2.1 (Pin_1)
- new net +5V: J2.10 (Pin_10), R1.1, R2.1, R3.1, R4.1, R5.1
- new net -5V: J2.11 (Pin_11)
- new net BD0: U13.9 (D0), U3.18 (B0), U5.33 (D0), U7.14 (D0), U8.14 (D0)
- new net BD1: U13.10 (D1), U3.17 (B1), U5.32 (D1), U7.13 (D1), U8.13 (D1)
- new net BD2: U13.11 (D2), U3.16 (B2), U5.31 (D2), U7.12 (D3), U8.12 (D3)
- new net BD3: U13.13 (D3), U3.15 (B3), U5.30 (D3), U7.11 (D3), U8.11 (D3)
- new net BD4: U13.14 (D4), U3.14 (B4), U5.29 (D4)
- new net BD5: U13.15 (D5), U3.13 (B5), U5.28 (D5)
- new net BD6: U13.16 (D6), U3.12 (B6), U5.27 (D6)
- new net BD7: U13.17 (D7), U3.11 (B7), U5.26 (D7)
- new net E: U5.37 (E)
- new net MBA: TP1. (D7), U10.15 (I2b)
- new net MVMA: TP1. (D7), U10.17 (I3b), U5.5 (VMA)
- new net MemR: R5.2, TP1. (D7), U5.3 (MR)
- new net R/~W: U5.34 (R/~{W})
- new net ~{MBA}: U5.7 (BA)
- no-connect marks 0 -> 6
Other:
- moved on the sheet: TP1

Commit message: wip
Parts:
- added J1, J2, J3: Conn_02x04_Odd_Even, symbol Connector_Generic:Conn_02x04_Odd_Even
- added TP2: TestPoint, symbol Connector:TestPoint
- added U11: MC6810, symbol 0.MekLib:MC6810
- added U12: 68A316E, symbol 0.MekLib:68A316E
- added U14: 74LS20, symbol 74xx:74LS20
- added U6: 74LS156, symbol 0.MekLib:74LS156
- added U9: User IO, symbol 0.MekLib:UserIO
- added Z2: 4.7K, symbol 0.MekLib:R_Array
Connections:
- net +5V: now also U4.10, U11.10 (SC0), U11.13 (CS3), U12.20 (~{S1}), U9.24 (+5), Z2.1
- net BA0: now also U6.36 (RS0), U11.23 (A0), U12. (A10)
- net BA1: now also U6.35 (RS1), U11.24 (A1), U12. (A10)
- net BA10: now also U12. (A10), U6.13 (A)
- net BA11: now also U6.3 (B)
- net BA12: now also U6.1 (1C)
- net BA13: now also U14.4
- net BA14: now also U14.2
- net BA15: now also U14.1
- net BA2: now also U4.9, U11.25 (A2), U12. (A10)
- net BA3: now also U11.26 (A3), U12. (A10)
- net BA4: now also U11.27 (A4), U12. (A10)
- net BA5: now also U11.28 (A5), U12. (A10)
- net BA6: now also U11.15 (~{CS5}), U12. (A10)
- net BA7: now also U6.22 (CS0), U11.11 (~{CS1}), U12. (A10)
- net BA8: now also U11.12 (~{CS2}), U12. (A10)
- net BA9: now also U12. (A10)
- net BD0: now also U6.33 (D0), U11.2 (D0), U12.9 (D0)
- net BD1: now also U6.32 (D1), U11.3 (D1), U12.10 (D1)
- net BD2: now also U6.31 (D2), U11.4 (D2), U12.11 (D2)
- net BD3: now also U6.30 (D3), U11.5 (D3), U12.13 (D3)
- net BD4: now also U6.29 (D4), U11.6 (D4), U12.14 (D4)
- net BD5: now also U6.28 (D5), U11.7 (D5), U12.15 (D5)
- net BD6: now also U6.27 (D6), U11.8 (D6), U12.16 (D6)
- net BD7: now also U6.26 (D7), U11.9 (D7), U12.17 (D7)
- net GND: now also U12.18 (~{S2}), U9.13 (GND)
- net MVMA: now also U4.2, U14.5
- net ~{IRQ}: now also J1.3 (Pin_3), J1.5 (Pin_5)
- net ~{NMI}: now also J1.1 (Pin_1), J1.7 (Pin_7)
- net ~{RESET}: now also U6.34 (~{RESET})
- net Ø2(E): now also U6.25 (ENABLE)
- net at U4.8: now also U6.24 (CS1)
- net at U4.1: now also TP2.1, U14.6, U6.14 (~{2G}), U6.2 (~{1G})
- net ~{OFF-BOARD}: now reaches U4.3
- net at U6.10 (PB0): now also U9.3 (PB0)
- net at U6.11 (PB1): now also U9.4 (PB1)
- net at U6.12 (PB2): now also U9.5 (PB2)
- net at U6.13 (PB3): now also U9.6 (PB3)
- net at U6.14 (PB4): now also U9.7 (PB4)
- net at U6.15 (PB5): now also U9.8 (PB5)
- net at U6.16 (PB6): now also U9.9 (PB6)
- net at U6.17 (PB7): now also U9.10 (PB7)
- net at U6.18 (CB1): now also U9.11 (CB1)
- net at U6.19 (CB2): now also U9.12 (CB2)
- net at U6.2 (PA0): now also U9.20 (PA0)
- net R~{W}: now reaches U6.21 (R/~{W})
- net ~{RAM/IO}: now reaches U6.23 (~{CS2})
- net ~{RAM/IO}: now also U6.10 (2Y1), Z2.9
- net at U6.3 (PA1): now also U9.19 (PA1)
- net at U6.37 (~{IRQB}): now also J1.6 (Pin_6), J1.8 (Pin_8)
- net at U6.38 (~{IRQA}): now also J1.2 (Pin_2), J1.4 (Pin_4)
- net at U6.39 (CA2): now also U9.21 (CA2)
- net at U6.4 (PA2): now also U9.18 (PA2)
- net at U6.40 (CA1): now also U9.22 (CA1)
- net at U6.5 (PA3): now also U9.17 (PA3)
- net at U6.6 (PA4): now also U9.16 (PA4)
- net at U6.7 (PA5): now also U9.15 (PA5)
- net at U6.8 (PA6): now also U9.1 (PA6)
- net at U6.9 (PA7): now also U9.2 (PA7)
- new net: J3.2 (Pin_2), J3.4 (Pin_4), J3.6 (Pin_6), J3.8 (Pin_8)
- new net: J2.1 (Pin_1), J2.3 (Pin_3), J2.5 (Pin_5), J2.7 (Pin_7)
- new net E8xx: J3.5 (Pin_5), U6.11 (2Y2), Z2.8
- new net ECxx: J3.7 (Pin_7), U6.12 (2Y3), Z2.7
- new net F0xx: J2.6 (Pin_6), U6.7 (Y10), Z2.6
- new net F4xx: J2.8 (Pin_8), U6.6 (1Y1), Z2.5
- new net F8xx: J2.4 (Pin_4), J3.3 (Pin_3), U6.5 (1Y2), Z2.4
- new net FCxx: J2.2 (Pin_2), J3.1 (Pin_1), U6.4 (1Y3), Z2.2
- new net ~{URAM}: U6.9 (2Y0), Z2.10
Other:
- moved on the sheet: C1, C2, J2, R1, R2, R3, R4, R5, TP1, U10A, U13A, U1A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
